Commit message: Restructure dual-arm FR3 onto a single controller_manager
The dual-arm config previously ran two namespaced controller_managers
(/left, /right). The stock MoveIt Pro teleop/jog behaviors hardcode
/controller_manager and /{controller}/command, so they cannot drive a
namespaced setup, and the namespaced control nodes never received the
SRDF (jog controllers failed on_configure). Mirror the known-good
dual_arm_sim wiring instead: a single un-namespaced controller_manager,
launched by the Agent, fed one combined URDF + SRDF + kinematics, with
left_/right_-prefixed controllers.

Control / hardware:
- description/franka.urdf.xacro: emit one ros2_control system per arm
  (left_/right_FrankaHardwareInterface) from a single combined URDF;
  use_fake_hardware arg selects mock vs real.
- config/control/franka_ros2_control.yaml: new single combined controller
  yaml (replaces the per-arm left_/right_ yamls). Combined 14-joint JTC
  (allow_partial_joints_goal + allow_nonzero_velocity_at_trajectory_end),
  per-arm JVC/VFC, franka_robot_state_broadcasters (arm_prefix/robot_type,
  not arm_id), and unprefixed UI shim controllers so the teleop UI's
  hardcoded param reads resolve (avoids the rosapi clock-type crash).
- config/config.yaml: single CM (launch_control_node: True,
  manage_controllers: True), startup controller lists, real-hardware
  defaults (simulated: False, use_fake_hardware: "false", JTC effort).

Teleop:
- config/moveit/franka.srdf: tip manipulator chains at *_grasp_link and
  repoint end-effectors at the *_manipulator groups so pose-jog and the
  interactive marker work.
- config/moveit/joint_jog.yaml: use the left_/right_ prefixed JVCs.
- objectives/teleoperate.xml: reference the core Request Teleoperation
  subtree, un-namespaced, initial_teleop_mode=3, no blackboard seeding;
  delete the vendored namespaced request_teleoperation.xml.

Grippers (real hardware): the FR3 grippers are libfranka action servers,
not ros2_control controllers, so rewrite robot_drivers_to_persist.launch.py
to launch one franka_gripper node per arm (left/right namespaces) and wire
it back via hardware.robot_driver_persist_launch_file. Delete the obsolete
per-arm left_/right_franka.launch.py.

Mock validated end-to-end (all teleop modes, both arms). Real hardware is
configured but untested; mock<->real requires manual edits to simulated,
use_fake_hardware, and the JTC command_interfaces.

Co-Authored-By: Claude Opus 4.8 (1M context) <noreply@anthropic.com>

File: src/franka_dual_arm_hw/description/franka.urdf.xacro (robot description, xacro)
@@ -5,4 +5,8 @@
   <xacro:arg name="ee_id" default="franka_hand" />
   <xacro:arg name="rpy_ee" default="0 0 -0.785" />
+  <!-- MOCK HARDWARE: default true loads mock_components/GenericSystem for both arms
+       (no robot/FCI needed). Set to false (via config.yaml urdf_params) to drive the
+       real dual FR3 with two franka_hardware/FrankaHardwareInterface systems. -->
+  <xacro:arg name="use_fake_hardware" default="true" />
   <!-- Load Franka robot -->
   <xacro:include filename="$(find franka_description)/robots/common/franka_robot.xacro"/>
@@ -14,5 +18,7 @@
   </joint>
   <!-- franka_description 2.7.1 selects joint_limits/inertials/kinematics/dynamics
-       internally from robot_type; they are no longer passed as macro params. -->
+       internally from robot_type; they are no longer passed as macro params.
+       ros2_control="true" emits one <ros2_control> system per arm (left_/right_),
+       both loaded by the single un-namespaced controller_manager. -->
   <xacro:franka_robot robot_type="fr3"
                       gazebo="false"
@@ -21,7 +27,7 @@
                       ee_id="$(arg ee_id)"
                       with_sc="false"
-                      ros2_control="false"
+                      ros2_control="true"
                       robot_ip="$(arg right_robot_ip)"
-                      use_fake_hardware="false"
+                      use_fake_hardware="$(arg use_fake_hardware)"
                       fake_sensor_commands="false"
                       gazebo_effort="false"
@@ -30,8 +36,9 @@
                       connected_to= "right_mount">
   </xacro:franka_robot>
-  <link name="grasp_link" />
-  <joint name="grasp_link_joint" type="fixed">
-     <parent link="world"/>
-     <child link = "grasp_link"/>
+  <!-- This link aligns the axes of the grasp frame to our required convention for motion planning tasks. -->
+  <link name="right_grasp_link" />
+  <joint name="right_grasp_link_joint" type="fixed">
+     <parent link="right_fr3_hand_tcp"/>
+     <child link = "right_grasp_link"/>
      <origin xyz="0 0 0" rpy="0 0 -1.5708"/>
   </joint>
@@ -49,7 +56,7 @@
                       ee_id="$(arg ee_id)"
                       with_sc="false"
-                      ros2_control="false"
+                      ros2_control="true"
                       robot_ip="$(arg left_robot_ip)"
-                      use_fake_hardware="false"
+                      use_fake_hardware="$(arg use_fake_hardware)"
                       fake_sensor_commands="false"
                       gazebo_effort="false"
@@ -58,8 +65,8 @@
                       connected_to= "left_mount">
   </xacro:franka_robot>
-    <!-- This link aligns the axes of the grasp frame to our required convention for motion planning tasks. -->
+   <!-- This link aligns the axes of the grasp frame to our required convention for motion planning tasks. -->
    <link name="left_grasp_link" />
    <joint name="left_grasp_link_joint" type="fixed">
-      <parent link="world"/>
+      <parent link="left_fr3_hand_tcp"/>
       <child link = "left_grasp_link"/>
       <origin xyz="0 0 0" rpy="0 0 -1.5708"/>
