Commit message: Root the Mobile FR3 Duo at odom with drifting simulated odometry
Both mobile packages now use world -> map (fixed) -> odom -> planar joints
-> base_link, with the URDF rooted at odom. It runs on MoveIt Pro 10.1.0
and main.

mobile_fr3_duo_mock:
- launch/frames.launch.py publishes world -> map and map -> odom as fixed
  identities, because mock hardware has no localization.
- The MuJoCo hardware settings (scene, package, keyframe, object TF,
  ground-truth odometry topic and frame, base link name) are xacro
  arguments, defaulting to mobile_fr3_duo_sim's values.

mobile_fr3_duo_sim:
- The simulator publishes the true base pose only as a message on
  /ground_truth/odom (frame mj_world) and publishes no base TF.
- script/odometry_joint_state_publisher.py is the only publisher of the
  planar joints and /odom, with drift that grows with distance and turn.
  Drift is on by default; the odometry_drift launch argument turns it off.
- joint_state_broadcaster lists every joint except the planar ones, so the
  true planar values stay off /joint_states.
- base_twist_to_planar.py uses the true heading from ground truth.
- The launch publishes world -> map and world -> mj_world; AMCL keeps
  map -> odom. odom_twist_to_base.py is replaced by the odometry bridge.
- Tests for the odometry and cmd_vel bridges.

File: src/mobile_fr3_duo_mock/description/mobile_fr3_duo.urdf.xacro (robot description, xacro)
@@ -2,18 +2,21 @@
 <robot xmlns:xacro="http://www.ros.org/wiki/xacro" name="mobile_fr3_duo">
   <xacro:arg name="hardware_interface" default="mock"/>
+  <!-- MuJoCo settings, used when hardware_interface is mujoco. A child config overrides them through urdf_params. -->
   <xacro:arg name="mujoco_model" default="mjcf/scene.xml"/>
+  <xacro:arg name="mujoco_model_package" default="mobile_fr3_duo_sim"/>
+  <xacro:arg name="mujoco_keyframe" default="default"/>
   <xacro:arg name="mujoco_viewer" default="false"/>
+  <xacro:arg name="publish_object_tf" default="true"/>
+  <xacro:arg name="ground_truth_odom_topic" default="/ground_truth/odom"/>
+  <xacro:arg name="ground_truth_odom_frame" default="mj_world"/>
+  <xacro:arg name="base_link_name" default="base_link"/>
   <xacro:include filename="$(find franka_description)/robots/mobile_fr3_duo_v0_2/mobile_fr3_duo_v0_2.xacro"/>
-  <link name="world"/>
-  <joint name="base_joint" type="fixed">
-    <parent link="world"/>
-    <child link="base"/>
-  </joint>
-  <!-- Planar base pose (x, y, yaw) as joints between the fixed base and the robot's base_link -->
-  <link name="base"/>
+  <!-- Frames: world -> map (fixed) -> odom -> planar joints -> base_link. The URDF starts at odom. -->
+  <!-- world -> map and map -> odom come from the launch files; the planar joints are odom -> base_link. -->
+  <link name="odom"/>
   <link name="virtual_x"/>
   <link name="virtual_y"/>
   <joint name="planar_x" type="prismatic">
-    <parent link="base"/>
+    <parent link="odom"/>
     <child link="virtual_x"/>
     <axis xyz="1 0 0"/>
@@ -41,5 +44,5 @@
     reduced_version="false"
     description_pkg="franka_description"
-    connected_to="base"
+    connected_to="odom"
     use_arms="true"
     no_prefix="false"
@@ -73,5 +76,13 @@
   <xacro:if value="${'$(arg hardware_interface)' == 'mujoco'}">
     <xacro:include filename="$(find mobile_fr3_duo_sim)/description/mobile_fr3_duo_mujoco.ros2_control.xacro"/>
-    <xacro:mobile_fr3_duo_mujoco_ros2_control mujoco_model="$(arg mujoco_model)" mujoco_viewer="$(arg mujoco_viewer)"/>
+    <xacro:mobile_fr3_duo_mujoco_ros2_control
+      mujoco_model="$(arg mujoco_model)"
+      mujoco_model_package="$(arg mujoco_model_package)"
+      mujoco_keyframe="$(arg mujoco_keyframe)"
+      mujoco_viewer="$(arg mujoco_viewer)"
+      publish_object_tf="$(arg publish_object_tf)"
+      ground_truth_odom_topic="$(arg ground_truth_odom_topic)"
+      ground_truth_odom_frame="$(arg ground_truth_odom_frame)"
+      base_link_name="$(arg base_link_name)"/>
   </xacro:if>
 </robot>

File: src/mobile_fr3_duo_sim/description/mobile_fr3_duo_mujoco.ros2_control.xacro (robot description, xacro)
@@ -1,5 +1,9 @@
 <?xml version="1.0"?>
 <robot xmlns:xacro="http://www.ros.org/wiki/xacro">
-  <xacro:macro name="mobile_fr3_duo_mujoco_ros2_control" params="mujoco_model mujoco_viewer">
+  <!-- MujocoSystem takes the joints and actuators from the MJCF, so none are listed here. -->
+  <xacro:macro
+    name="mobile_fr3_duo_mujoco_ros2_control"
+    params="mujoco_model mujoco_model_package mujoco_keyframe mujoco_viewer publish_object_tf
+            ground_truth_odom_topic ground_truth_odom_frame base_link_name">
     <ros2_control name="mobile_fr3_duo" type="system">
       <sensor name="lidar_front">
@@ -12,20 +16,21 @@
         <plugin>picknik_mujoco_ros/MujocoSystem</plugin>
         <param name="mujoco_model">${mujoco_model}</param>
-        <param name="mujoco_model_package">mobile_fr3_duo_sim</param>
+        <param name="mujoco_model_package">${mujoco_model_package}</param>
         <param name="mujoco_viewer">${mujoco_viewer}</param>
-        <param name="mujoco_keyframe">default</param>
+        <param name="mujoco_keyframe">${mujoco_keyframe}</param>
         <param name="render_publish_rate">10</param>
         <param name="point_cloud_publish_rate">10</param>
         <param name="tf_publish_rate">60</param>
         <param name="lidar_publish_rate">10</param>
-        <!-- mj_world -> map -> odom -> world come from static transforms in
-             launch/additional_driver_nodes.launch.py, so the plugin must not parent world. -->
+        <!-- The URDF root odom is not a MuJoCo body, so the base body is named explicitly. -->
+        <param name="base_link_name">${base_link_name}</param>
+        <!-- world -> mj_world comes from launch/additional_driver_nodes.launch.py, so the plugin must not publish it. -->
         <param name="publish_mj_world_tf">false</param>
-        <!-- /odom for Nav2 (ground truth). No TF: robot_state_publisher owns the chain to base_link. -->
+        <param name="publish_object_tf">${publish_object_tf}</param>
+        <!-- Ground truth as a message only: the odometry bridge adds drift and publishes the planar joints. -->
         <param name="publish_odom">true</param>
-        <!-- Raw: the plugin reports the twist in the odom frame. odom_twist_to_base.py
-             rotates it into base_link and republishes /odom. -->
-        <param name="odom_topic">/mujoco/odom</param>
-        <param name="odom_frame">odom</param>
+        <param name="odom_topic">${ground_truth_odom_topic}</param>
+        <!-- The frame the true pose is in. MoveIt Pro requires it to differ from the URDF root. -->
+        <param name="odom_frame">${ground_truth_odom_frame}</param>
         <param name="odom_child_frame">base_link</param>
         <param name="odom_rate">50</param>
