Commit message: Navigate the Mobile FR3 Duo mock with Nav2, arms stowed before every drive
mobile_fr3_duo_mock now runs Nav2 on the room map: launch/navigation.launch.py
starts the map server and Nav2 with params/nav2_params.yaml (static map only,
fixed map -> odom), script/joint_state_odometry.py publishes /odom from the
planar joints, and base_twist_to_planar.py drives the planar joints through
base_jgvc. The base jog controllers now command velocity too, and base_jtc
is gone, so a jog and Nav2 hand the base over cleanly. The room map, the
twist bridge and the navigation Objectives move from mobile_fr3_duo_sim to
the mock; "Move Base to Ready" drives with Nav2 in both packages.

mobile_fr3_duo_sim reuses the mock's navigation launch with AMCL, its true
heading for the bridge, and a small Nav2 overlay for AMCL and the laser
obstacle layers (mappings merge, lists replace).

Every navigation Objective first runs "Stow Arms for Navigation", which
moves both arms and the spine to the Stow waypoint. The Nav2 footprint in
both costmaps covers the robot in that pose, taken from the MuJoCo model's
geometry with a margin, and the MPPI cost critic now checks the full
footprint.

File: src/mobile_fr3_duo_mock/description/mobile_fr3_duo_mock.ros2_control.xacro (robot description, xacro)
@@ -6,4 +6,14 @@
       <state_interface name="position">
         <param name="initial_value">${initial_position}</param>
+      </state_interface>
+      <state_interface name="velocity"/>
+    </joint>
+  </xacro:macro>
+  <!-- The base controllers (Nav2's base_jgvc and the base jogs) command velocity. -->
+  <xacro:macro name="mobile_fr3_duo_mock_planar_joint" params="name">
+    <joint name="${name}">
+      <command_interface name="velocity"/>
+      <state_interface name="position">
+        <param name="initial_value">0.0</param>
       </state_interface>
       <state_interface name="velocity"/>
@@ -34,7 +44,7 @@
         <param name="calculate_dynamics">true</param>
       </hardware>
-      <xacro:mobile_fr3_duo_mock_commanded_joint name="planar_x"/>
-      <xacro:mobile_fr3_duo_mock_commanded_joint name="planar_y"/>
-      <xacro:mobile_fr3_duo_mock_commanded_joint name="planar_theta"/>
+      <xacro:mobile_fr3_duo_mock_planar_joint name="planar_x"/>
+      <xacro:mobile_fr3_duo_mock_planar_joint name="planar_y"/>
+      <xacro:mobile_fr3_duo_mock_planar_joint name="planar_theta"/>
       <xacro:mobile_fr3_duo_mock_commanded_joint name="franka_spine_vertical_joint"/>
       <xacro:mobile_fr3_duo_mock_arm_joints prefix="left"/>
